File: Previous Versions/Rev1-0/electronics-function-generator.sch (KiCad schematic (older format))
At the start: 23 parts

Commit message: Rev 2-0: revert passive values back to XR2206 app notes.
Parts:
- removed C?: 10uF, Capacitor_SMD:C_1206_3216Metric_Pad1.33x1.80mm_HandSolder, symbol Device:C
- added C?: 0.1u, Capacitor_SMD:C_1206_3216Metric_Pad1.33x1.80mm_HandSolder, symbol Device:C
- C?: value 1uF -> 100u
- C?: value 1uF -> 10u
- R?: value 10K -> 1K
Connections:
- net +12V: now also C?.1
- net Amplitude: now also RV?.2
- net GND: now also C?.2
- net at R?.1, R?.2, RV?.3: no longer RV?.2
Other:
- note added: "1-0"
- note added: "9 April 2021"
- note removed: "10 April 2021"
- note removed: "2-0"
- note removed: "2-0: Revert passive values back to XR2206 app notes."
- moved on the sheet: C?, J?, JP?, R?
